Commit message: Robot can no longer drive through walls: box chassis collision
The chassis collision used the decorative STL trimesh; Gazebo/ODE trimesh
contacts are unreliable and let the robot push through the (properly
collided) walls. Collision is now a chassis-sized box - verified by
driving full speed into the east wall for 45 s: robot pins at x=5.81
against the wall face at x=5.92.

Also wrap robot_description in ParameterValue(value_type=str) in
rsp.launch.py so URDF content can never abort the launch as bad YAML.

Co-Authored-By: Claude Fable 5 <noreply@anthropic.com>

File: src/yoru_base/description/robot_core.xacro (robot description, xacro)
@@ -50,9 +50,11 @@
             <material name="yellow"/>
         </visual>
+        <!-- Collision is a simple box (not the decorative mesh) because
+             Gazebo/ODE trimesh contacts are unreliable and let the robot
+             push through walls. Box-vs-box contacts are solid. -->
         <collision>
-            <origin xyz="${chassis_length/2} 0 ${chassis_height/2}"/>
+            <origin xyz="${chassis_length/2} 0 0.05"/>
             <geometry>
-                <mesh filename="package://yoru_base/meshes/body_bot.stl"
-                      scale="0.001 0.001 0.001"/>
+                <box size="${chassis_length} ${chassis_width} 0.1"/>
             </geometry>
         </collision>
