Commit message: Real hardware bring-up: Nano Every motor bridge replaces GPIO driver
The robot's actual motor chain is Pi -> Arduino Nano Every -> L298N
(ROSArduinoBridge-standard wiring), not L298N on Pi GPIO:

- firmware/yoru_motor_bridge: ROSArduinoBridge port for the Nano Every
  (attachInterrupt encoders instead of ATmega328 PCINT ISRs); encoder
  sign flipped to match this chassis, bench-verified
- arduino_driver_node: serial bridge (57600 baud) with kinematics +
  odometry, same topic contract as the old l298n_driver_node
- measured constants: enc_counts_per_rev 3166 (hand-calibrated),
  wheel radius 0.0325m, wheel track 0.32m - applied to real config,
  URDF and sim so they match the physical robot
- rplidar launch: A1 port by-path + 115200 baud

Verified on the robot: /scan 6.8Hz, IMX477 camera 17.3Hz, /odom
17.6Hz, slam_toolbox mapping, 2s drive test odom +0.233m straight.

Co-Authored-By: Claude Fable 5 <noreply@anthropic.com>

File: src/yoru_base/description/gazebo_control.xacro (robot description, xacro)
@@ -6,6 +6,6 @@
             <left_joint>left_wheel_joint</left_joint>
             <right_joint>right_wheel_joint</right_joint>
-            <wheel_separation>0.297</wheel_separation>
-            <wheel_diameter>0.066</wheel_diameter>
+            <wheel_separation>0.32</wheel_separation>
+            <wheel_diameter>0.065</wheel_diameter>
             <!-- Limits -->
             <max_wheel_torque>200</max_wheel_torque>

File: src/yoru_base/description/robot_core.xacro (robot description, xacro)
@@ -8,9 +8,10 @@
     <xacro:property name="chassis_height" value="0"/>
     <xacro:property name="chassis_mass" value="1.0"/>
-    <xacro:property name="wheel_radius" value="0.033"/>
-    <xacro:property name="wheel_thickness" value="0.026"/>
+    <xacro:property name="wheel_radius" value="0.0325"/>
+    <xacro:property name="wheel_thickness" value="0.025"/>
     <xacro:property name="wheel_mass" value="0.05"/>
     <xacro:property name="wheel_offset_x" value="0.226"/>
-    <xacro:property name="wheel_offset_y" value="0.1485"/>
+    <!-- measured on the real chassis 2026-07-07: 32cm track -->
+    <xacro:property name="wheel_offset_y" value="0.16"/>
     <xacro:property name="wheel_offset_z" value="0.01"/>
     <xacro:property name="caster_wheel_radius" value="0.01"/>

Commit message: Recalibrate for new wheels/encoders: 1320 counts/rev, 87mm wheels
New hardware (2026-07-29): encoders 1320 counts per wheel revolution,
wheels 87mm diameter (0.0435m radius) x 40mm thick. Updated everywhere:
arduino_driver_node + yoru_real.yaml (enc_counts_per_rev, wheel_radius),
robot_core.xacro (radius + thickness), my_controllers.yaml (sim radius),
gazebo_control.xacro (wheel_diameter). Wheel track unchanged at 0.32m.

Co-Authored-By: Claude Opus 4.8 <noreply@anthropic.com>

File: src/yoru_base/description/gazebo_control.xacro (robot description, xacro)
@@ -7,5 +7,5 @@
             <right_joint>right_wheel_joint</right_joint>
             <wheel_separation>0.32</wheel_separation>
-            <wheel_diameter>0.065</wheel_diameter>
+            <wheel_diameter>0.087</wheel_diameter>
             <!-- Limits -->
             <max_wheel_torque>200</max_wheel_torque>

File: src/yoru_base/description/robot_core.xacro (robot description, xacro)
@@ -8,6 +8,6 @@
     <xacro:property name="chassis_height" value="0"/>
     <xacro:property name="chassis_mass" value="1.0"/>
-    <xacro:property name="wheel_radius" value="0.0325"/>
-    <xacro:property name="wheel_thickness" value="0.025"/>
+    <xacro:property name="wheel_radius" value="0.0435"/>
+    <xacro:property name="wheel_thickness" value="0.04"/>
     <xacro:property name="wheel_mass" value="0.05"/>
     <xacro:property name="wheel_offset_x" value="0.226"/>
